Commit message: added no-gui launch files for robot

File: r2_gazebo/urdf/gazebo_plugins/r2.transmissions.xacro (robot description, xacro)
@@ -5,5 +5,7 @@
      <transmission name="${part}_j${joint}_trans">
        <type>transmission_interface/SimpleTransmission</type>
-       <joint name="${part}/joint${joint}"/>
+       <joint name="${part}/joint${joint}">
+         <hardwareInterface>EffortJointInterface</hardwareInterface>
+       </joint>
        <actuator name="${part}_j${joint}_motor">
          <hardwareInterface>EffortJointInterface</hardwareInterface>

File: r2_gazebo/urdf/gazebo_plugins/r2_legs.transmissions.xacro (robot description, xacro)
@@ -5,5 +5,7 @@
      <transmission name="${part}_j${joint}_trans">
        <type>transmission_interface/SimpleTransmission</type>
-       <joint name="${part}/joint${joint}"/>
+       <joint name="${part}/joint${joint}">
+         <hardwareInterface>EffortJointInterface</hardwareInterface>
+       </joint>
        <actuator name="${part}_j${joint}_motor">
          <hardwareInterface>EffortJointInterface</hardwareInterface>
