Commit message: Specify hardwareInterface inside joint tags
This is needed for ros-control on indigo.
See the following for more info:
https://github.com/ros-controls/ros_control/issues/177
https://github.com/ros-simulation/gazebo_ros_demos/pull/4

File: r2_gazebo/xacro/gazebo_plugins/r2.transmissions.xacro (robot description, xacro)
@@ -5,5 +5,7 @@
      <transmission name="${part}_trans">
        <type>transmission_interface/SimpleTransmission</type>
-       <joint name="${part}"/>
+       <joint name="${part}">
+         <hardwareInterface>EffortJointInterface</hardwareInterface>
+       </joint>
        <actuator name="${part}_motor">
          <hardwareInterface>EffortJointInterface</hardwareInterface>

File: r2_gazebo/xacro/gazebo_plugins/r2_legs.transmissions.xacro (robot description, xacro)
@@ -5,5 +5,7 @@
      <transmission name="${part}_trans">
        <type>transmission_interface/SimpleTransmission</type>
-       <joint name="${part}"/>
+       <joint name="${part}">
+         <hardwareInterface>EffortJointInterface</hardwareInterface>
+       </joint>
        <actuator name="${part}_motor">
          <hardwareInterface>EffortJointInterface</hardwareInterface>
